Commit message: config to moveit: ready to use with python

File: catkin_ws/src/KUKA_5/kr5_gazebo/urdf/gazebo.xacro (robot description, xacro)
@@ -9,5 +9,5 @@
     <parent link="world"/>
     <child link="base_link"/>
-    <origin xyz="0.0 0.0 0.0" rpy="0.0 0.0 0.0" />
+    <origin xyz="0.0 0.0 0.0" rpy="0.0 0.0 -1.5707" />
   </joint>
 </robot>
